File: PCB/HASwitchPlate.kicad_pcb (KiCad board)
At the start: 2 copper layers, 60 x 40 mm, 11 parts, among them J1 Screw Term., J2 XH2.54-4P, J3 Breakout, U1 IRM-03-5, U2 WeMos_mini

Commit message: PCB v0.06
Parts:
- moved REF*** 1.86 mm to (136.2, 119.0)
- moved G*** 0.51 mm to (137.0, 120.2)
Other:
- outline, holes or cut-outs redrawn
- board text added: "AC"
- board text added: "L"
- board text added: "N"
- board text added: "v0.06"
- board text removed: "v0.04"

Commit message: HASP v0.35
Parts:
- removed the REF** at (102.0, 102.0)
- removed the REF** at (158.0, 102.0)
- removed the REF** at (102.0, 138.0)
- removed REF***: OSHW-Logo_19x20mm_SilkScreen, Symbols:OSHW-Logo_19x20mm_SilkScreen
- added Q1: S8050, Package_TO_SOT_THT:TO-92L_HandSolder, F.Cu at (152.1, 104.8)
- added R1: 1k, Resistor_THT:R_Axial_DIN0207_L6.3mm_D2.5mm_P10.16mm_Horizontal, F.Cu at (151.9, 118.7)
- added REF**: MountingHole_2.2mm_M2, HASwitchPlate:MountingHole_2.2mm_M2, F.Cu at (101.8, 101.6)
- added REF** (x2): MountingHole_2.2mm_M2, HASwitchPlate:MountingHole_2.2mm_M2, F.Cu at (101.8, 101.7)
- added REF**: OSHW-Logo_11.4x12mm_SilkScreen, Symbol:OSHW-Logo_11.4x12mm_SilkScreen, F.Cu at (135.3, 130.5)
- added REF**: KiCad-Logo2_12mm_SilkScreen, Symbol:KiCad-Logo2_12mm_SilkScreen, B.Cu at (134.0, 125.7)
- added REF**: OSHW-Logo_11.4x12mm_SilkScreen, Symbol:OSHW-Logo_11.4x12mm_SilkScreen, B.Cu at (134.5, 106.6)
- added U3: SLC03-series, HASwitchPlate:ACDC-Converter_MeanWell-SLC03-series, F.Cu at (147.0, 135.7)
- moved G*** 8.01 mm to (137.3, 112.2)
- moved J2 2.57 mm to (157.8, 110.8)
- moved G*** 0.31 mm to (110.8, 121.6)
Connections:
- J2 pad 1: /GND -> /LCD_GND
- U2 pad 12: (no net) -> Net-(U2-Pad12)
- U2 pad 13: (no net) -> Net-(R1-Pad1)
- U2 pad 4: (no net) -> Net-(U2-Pad4)
- U2 pad 7: (no net) -> Net-(U2-Pad7)
- U2 pad 8: (no net) -> Net-(U2-Pad8)
- U2 pad 9: (no net) -> Net-(U2-Pad9)
Routing:
- net Net-(R1-Pad1): track 0.00 -> 74.1 mm, vias 0 -> 1
- net /+5V: track 0.00 -> 30.1 mm
- net /AC_N: track 17.0 -> 0.00 mm
- net /AC_L: track 17.0 -> 0.00 mm
- net /LCD_GND: track 0.00 -> 16.6 mm, vias 0 -> 1
- net /LCD_CTL: track 0.00 -> 9.82 mm
- net /D8_DBG: track 35.0 -> 44.5 mm
- net /D0: track 22.3 -> 26.6 mm
- net /A0: track 18.7 -> 22.6 mm
- net /LCD_TX: track 65.9 -> 68.8 mm
- net /+3.3V: track 34.5 -> 36.3 mm
- net /LCD_RX: track 36.2 -> 37.9 mm, vias 0 -> 1
- added copper zone on B.Cu, net /+5V
- added copper zone on B.Cu, net /AC_L
- added copper zone on F.Cu, net /AC_L
- added copper zone on B.Cu, net /AC_N
- added copper zone on F.Cu, net /AC_N
- added copper zone on F.Cu, net /GND
- removed copper zone on F.Cu, net /+5V
- removed copper zone on B.Cu, net /GND
Other:
- outline, holes or cut-outs redrawn
- board text added: "DC+"
- board text added: "DC-"
- board text added: "HASwitchPlate v1.0"
- board text added: "LCD"
- board text added: "NPN"
- board text added: "R1 1k"
- board text added: "SLC03x"
- board text added: "http://haswitchplate.com"
- board text added: "v1.0"
- board text removed: "AC"
- board text removed: "L"
- board text removed: "N"
- board text removed: "github.com/aderusha/HASwitchPlate"
- board text removed: "v0.06"
